File: spiresplit60/spiresplit60.kicad_pcb (KiCad board)
At the start: 2 copper layers, 200 parts

Commit message: Placed all switches and switch diodes
Parts:
- removed K_0, K_1, K_2, K_3, K_4, K_5, K_6, K_7, K_8, K_9, K_A, K_B, K_C, K_CBRAC, K_COMMA, K_D, K_DOT, K_E, K_EQUAL, K_EXTRA1A, K_F, K_G, K_H, K_I, K_J, K_K, K_L, K_M, K_MENU, K_MINUS, K_MOD1, K_N, K_O, K_OBRAC, K_P, K_Q, K_QUOTE, K_R, K_S, K_SEMIC, K_SLASH, K_SPACE, K_T, K_U, K_V, K_W, K_WIN, K_WIN1, K_X, K_Y, K_Z, K_`: KEYSW, MX_Alps_Hybrid:MX-1U-NoLED
- removed K_ALT1, K_BSLSH, K_CTRL, K_CTRL1, K_SPACE1, K_SPACE2, K_SPACE3, K_SPACE4, K_TAB: KEYSW, MX_Alps_Hybrid:MX-1.5U-NoLED
- removed K_BACKSPACE, K_ENTER, K_SHIFT: KEYSW, MX_Alps_Hybrid:MX-2U-NoLED
- removed K_CAPS, K_SHIFT1: KEYSW, MX_Alps_Hybrid:MX-1.75U-NoLED
- D67: footprint kbd:CherryMX_Choc_1u -> Diode_SMD:D_SOD-123
- moved MX_1 334.0 mm to (-29.4, 9.53)
- moved MX_2 315.3 mm to (-10.3, 9.53)
- moved D54 312.1 mm to (282.6, 72.2)
- moved D41 296.9 mm to (273.1, 53.2)
- moved MX_3 294.3 mm to (8.73, 9.53)
- moved D14 293.4 mm to (273.1, 14.3)
- moved D28 292.0 mm to (277.0, 34.1)
- moved D53 287.0 mm to (256.4, 72.2)
- moved D65 285.8 mm to (278.6, 91.3)
- moved D27 284.5 mm to (254.0, 34.1)
- moved MX_\1 280.1 mm to (271.5, 28.6)
- moved MX_ESC1 279.5 mm to (-48.4, 9.53)
- moved MX_4 278.8 mm to (27.8, 9.53)
- moved D64 271.9 mm to (254.0, 91.3)
- moved D13 271.0 mm to (244.5, 14.3)
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- renumbered MX_M2 to MX_M1, MX_M1 to MX_MACRO1

Commit message: idek what is going on with the lib
Parts:
- added J1: AudioJack3, Connector_Audio:Jack_3.5mm_Ledino_KB3SPRS_Horizontal, F.Cu at (122.2, 159.5)
- added J2: AudioJack3, Connector_Audio:Jack_3.5mm_Ledino_KB3SPRS_Horizontal, F.Cu at (122.2, 174.1)
- added SW1: SW_Push, Button_Switch_SMD:SW_SPST_TL3342, F.Cu at (116.7, 180.2)
- added SW2: SW_Push, Button_Switch_SMD:SW_SPST_TL3342, F.Cu at (126.2, 180.2)
- added U1: ProMicro, kbd:ProMicro_v3, F.Cu at (21.4, 134.9)
- added U2: ProMicro, kbd:ProMicro_v3, F.Cu at (102.4, 166.5)
- D1, D10, D11, D12, D13, D14, D15, D16, D17, D18, D19, D2, D20, D21, D22, D23, D24, D25, D26, D27, D28, D29, D3, D30, D31, D32, D33, D34, D35, D36, D37, D38, D39, D4, D40, D41, D42, D43, D44, D45, D46, D47, D48, D49, D5, D50, D51, D52, D53, D54, D55, D56, D57, D58, D59, D6, D60, D61, D62, D63, D64, D65, D66, D67, D7, D8, D9: moved to B.Cu
- MX_'1, MX_,1, MX_-1, MX_.1, MX_/1, MX_0, MX_1, MX_2, MX_3, MX_4, MX_5, MX_6, MX_7, MX_8, MX_9, MX_;1, MX_=1, MX_A1, MX_B1, MX_BS1, MX_C1, MX_CAPS1, MX_D1, MX_E1, MX_ENTER1, MX_ESC1, MX_EXTRA1, MX_F1, MX_G1, MX_H1, MX_I1, MX_J1, MX_K1, MX_L1, MX_LALT1, MX_LCTRL1, MX_LSHIFT1, MX_LWIN1, MX_M1, MX_MACRO1, MX_MOD1, MX_MOD2, MX_N1, MX_O1, MX_P1, MX_Q1, MX_R1, MX_RALT1, MX_RCTRL1, MX_RSHIFT1, MX_RWIN1, MX_S1, MX_SPACE1, MX_SPACE2, MX_SPACE3, MX_SPACE4, MX_T1, MX_TAB1, MX_U1, MX_V1, MX_W1, MX_X1, MX_Y1, MX_Z1, MX_[1, MX_\1, MX_]1: footprint kbd:CherryMX_Choc_1u -> keyswitches:SW_PG1350
- moved D66 16.2 mm to (51.6, 106.4), turned to 90 degrees
- moved D65 15.9 mm to (262.7, 92.1), turned to 270 degrees
- moved D19 15.1 mm to (29.4, 34.9), turned to 270 degrees
- moved D7 15.1 mm to (57.1, 15.9), turned to 270 degrees
- moved D4 15.1 mm to (0.79, 15.9), turned to 270 degrees
- moved D41 15.1 mm to (258.0, 53.9), turned to 270 degrees
- moved D54 15.1 mm to (267.5, 73.0), turned to 270 degrees
- moved D12 14.4 mm to (211.1, 15.9), turned to 270 degrees
- moved D10 14.4 mm to (173.0, 15.9), turned to 270 degrees
- moved D47 14.4 mm to (62.7, 73.0), turned to 270 degrees
- moved D44 14.4 mm to (5.56, 73.0), turned to 270 degrees
- moved D14 14.4 mm to (258.8, 15.8), turned to 270 degrees
- moved D11 14.4 mm to (192.1, 15.8), turned to 270 degrees
- moved D13 14.4 mm to (230.2, 15.8), turned to 270 degrees
- moved D9 14.4 mm to (154.0, 15.8), turned to 270 degrees
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Connections:
- net Net-(D1-Pad2) renamed Col1
- net Net-(D10-Pad2) renamed Col10
- net Net-(D21-Pad2) renamed Col14
- net Net-(D29-Pad2) renamed Row3
- net Net-(D35-Pad2) renamed Row8
- net Net-(D42-Pad2) renamed Row4
- net Net-(D48-Pad2) renamed Row9
- net Net-(D55-Pad2) renamed Row5
- net Net-(D60-Pad2) renamed Row10
- D15 pad 2: Net-(D15-Pad2) -> Row2
- D16 pad 2: Net-(D15-Pad2) -> Row2
- D17 pad 2: Net-(D15-Pad2) -> Row2
- D18 pad 2: Net-(D15-Pad2) -> Row2
- D19 pad 2: Net-(D15-Pad2) -> Row2
- D20 pad 2: Net-(D15-Pad2) -> Net-(D20-Pad2)
- MX_A1 pad 1: Net-(MX_1-Pad1) -> Net-(MX_2-Pad1)
- MX_B1 pad 1: Net-(MX_5-Pad1) -> Net-(MX_6-Pad1)
- MX_C1 pad 1: Net-(MX_3-Pad1) -> Net-(MX_4-Pad1)
- MX_D1 pad 1: Net-(MX_3-Pad1) -> Net-(MX_4-Pad1)
- MX_E1 pad 1: Net-(MX_3-Pad1) -> Net-(MX_4-Pad1)
- MX_F1 pad 1: Net-(MX_4-Pad1) -> Net-(MX_5-Pad1)
- MX_G1 pad 1: Net-(MX_5-Pad1) -> Net-(MX_6-Pad1)
- MX_I1 pad 1: Net-(MX_8-Pad1) -> Net-(MX_,1-Pad1)
- MX_MACRO1 pad 1: Net-(MX_'1-Pad1) -> Net-(MX_MACRO1-Pad1)
- MX_MOD1 pad 1: Net-(MX_5-Pad1) -> Net-(MX_6-Pad1)
- MX_MOD2 pad 1: Net-(MX_7-Pad1) -> Net-(MX_8-Pad1)
- MX_O1 pad 1: Net-(MX_,1-Pad1) -> Net-(MX_.1-Pad1)
- MX_P1 pad 1: Net-(MX_.1-Pad1) -> Net-(MX_-1-Pad1)
- MX_Q1 pad 1: Net-(MX_1-Pad1) -> Net-(MX_2-Pad1)
- MX_R1 pad 1: Net-(MX_4-Pad1) -> Net-(MX_5-Pad1)
- MX_RSHIFT1 pad 1: Net-(MX_'1-Pad1) -> Net-(MX_MACRO1-Pad1)
- MX_S1 pad 1: Net-(MX_2-Pad1) -> Net-(MX_3-Pad1)
- MX_SPACE1 pad 1: Net-(MX_3-Pad1) -> Net-(MX_4-Pad1)
- MX_SPACE2 pad 1: Net-(MX_4-Pad1) -> Net-(MX_5-Pad1)
- MX_SPACE3 pad 1: Net-(MX_8-Pad1) -> Net-(MX_7-Pad1)
- MX_T1 pad 1: Net-(MX_5-Pad1) -> Net-(MX_6-Pad1)
- MX_U1 pad 1: Net-(MX_7-Pad1) -> Net-(MX_8-Pad1)
- MX_V1 pad 1: Net-(MX_4-Pad1) -> Net-(MX_5-Pad1)
- MX_W1 pad 1: Net-(MX_2-Pad1) -> Net-(MX_3-Pad1)
- MX_X1 pad 1: Net-(MX_2-Pad1) -> Net-(MX_3-Pad1)
- MX_Y1 pad 1: Net-(MX_Y1-Pad1) -> Net-(MX_7-Pad1)
- MX_Z1 pad 1: Net-(MX_1-Pad1) -> Net-(MX_2-Pad1)
- MX_[1 pad 1: Net-(MX_-1-Pad1) -> Net-(MX_'1-Pad1)
- MX_]1 pad 1: Net-(MX_'1-Pad1) -> Net-(MX_MACRO1-Pad1)
Other:
- board text added: "WTF"

Commit message: Finished edge cuts
Parts:
- removed J1, J2: AudioJack3, Connector_Audio:Jack_3.5mm_Ledino_KB3SPRS_Horizontal
- added U3: TRRS, Keebio-Parts:TRRS-PJ-320A, F.Cu at (56.4, -3.97)
- added U4: TRRS, Keebio-Parts:TRRS-PJ-320A, F.Cu at (152.4, -3.97)
- MX_'1, MX_,1, MX_-1, MX_.1, MX_/1, MX_0, MX_1, MX_2, MX_3, MX_4, MX_5, MX_6, MX_7, MX_8, MX_9, MX_;1, MX_=1, MX_A1, MX_B1, MX_BS1, MX_C1, MX_CAPS1, MX_D1, MX_E1, MX_ENTER1, MX_ESC1, MX_EXTRA1, MX_F1, MX_G1, MX_H1, MX_I1, MX_J1, MX_K1, MX_L1, MX_LALT1, MX_LCTRL1, MX_LSHIFT1, MX_LWIN1, MX_M1, MX_MACRO1, MX_MOD1, MX_MOD2, MX_N1, MX_O1, MX_P1, MX_Q1, MX_R1, MX_RALT1, MX_RCTRL1, MX_RSHIFT1, MX_RWIN1, MX_S1, MX_SPACE1, MX_SPACE2, MX_SPACE3, MX_SPACE4, MX_T1, MX_TAB1, MX_U1, MX_V1, MX_W1, MX_X1, MX_Y1, MX_Z1, MX_[1, MX_\1, MX_]1: footprint keyswitches:SW_PG1350 -> Keebio-Parts:Kailh-PG1350-1u
- SW1, SW2: moved to B.Cu
- moved U2 237.5 mm to (290.5, 21.4)
- moved U1 144.2 mm to (-67.5, 21.4)
- moved SW1 105.0 mm to (42.9, 105.6)
- moved SW2 89.5 mm to (169.1, 101.6)
Other:
- board outline added: 378.6 x 118.3 mm
- board text removed: "WTF"
